Commit message: Examen Parte 2: Sensores RPLIDAR A3 Outdoor y Orbbec Astra S configurados

File: ros2_ws_mecanum/src/mi_robot_mecanum/urdf/mi_robot.urdf.xacro (robot description, xacro)
@@ -83,36 +83,31 @@
   <!-- TODO: link "lidar_link" (cilindro) con dimensiones y masa de la hoja de datos:
        visual, collision e inertial -->
-       <link name="lidar_link">
-        <visual>
-          <geometry><cylinder radius="0.076" length="0.041"/></geometry>
-           <origin xyz="0 0 0.02" rpy="0 0 0"/>
-           <material name="negro"><color rgba="0.1 0.1 0.1 1"/></material>
-        </visual>
-        <collision>
-          <origin xyz="0 0 0.02" rpy="0 0 0"/>
-          <geometry><cylinder radius="0.076" length="0.041"/></geometry>
-        </collision>
-        <inertial>
-          <origin xyz="0 0 0.02" rpy="0 0 0"/>
-          <mass value="0.19"/> <!-- Masa kg -->
-          <xacro:inercia_caja m="${chasis_masa}" x="${chasis_largo}" y="${chasis_ancho}" z="${chasis_alto}"/>
-       </inertial>
-        <inertial>
-        <mass value="0.19"/> <!-- Masa kg -->
-        <inertia ixx="0.0001" ixy="0" ixz="0" iyy="0.0001" iyz="0" izz="0.0001"/>
-        </inertial>
-        <visual><geometry><cylinder radius="0.076" length="0.041"/></geometry></visual>
-      </link>
+  <link name="lidar_link">
+  <visual>
+    <origin xyz="0 0 0.02" rpy="0 0 0"/>
+    <geometry><cylinder radius="0.038" length="0.041"/></geometry>
+    <material name="negro"><color rgba="0.1 0.1 0.1 1"/></material>
+  </visual>
+  <collision>
+    <origin xyz="0 0 0.02" rpy="0 0 0"/>
+    <geometry><cylinder radius="0.038" length="0.041"/></geometry>
+  </collision>
+  <inertial>
+    <origin xyz="0 0 0.02" rpy="0 0 0"/>
+    <mass value="0.19"/> <!-- Masa kg -->
+    <xacro:inercia_cilindro m="0.19" r="0.038" h="0.041"/>
+  </inertial>
+  </link>
   <!-- TODO: joint fijo "joint_lidar" base_link -> lidar_link en la posición de su variante -->
-      <joint name="lidar_joint" type="fixed">
-        <parent link="base_link"/>
-        <child link="lidar_link"/>
-        <origin xyz="0 0 0.02" rpy="0 0 0"/>
-      </joint>
+  <joint name="lidar_joint" type="fixed">
+    <parent link="base_link"/>
+    <child link="lidar_link"/>
+    <origin xyz="0.06 0 0.13" rpy="0 0 0"/>
+  </joint>
   <gazebo reference="lidar_link">
     <sensor name="rplidar_a3" type="gpu_lidar">
       <topic>/scan</topic>
-      <gz_frame_id>TODO</gz_frame_id>
-      <update_rate>TODO</update_rate>
+      <gz_frame_id>lidar_link</gz_frame_id>
+      <update_rate>5.0</update_rate> <!-- Barrido Variante F: 5 Hz -->
       <always_on>1</always_on>
       <visualize>true</visualize>
@@ -120,13 +115,13 @@
         <scan>
           <horizontal>
-            <samples>TODO</samples>          <!-- muestras por vuelta -->
+            <samples>2000</samples>          <!-- muestras por vuelta --> <!-- 10000 muestras/s (Outdoor) / 5 Hz = 2000 muestras -->
             <resolution>1</resolution>
-            <min_angle>TODO</min_angle>
-            <max_angle>TODO</max_angle>
+            <min_angle>-3.14159</min_angle>
+            <max_angle>3.14159</max_angle>
           </horizontal>
         </scan>
         <range>
-          <min>TODO</min>
-          <max>TODO</max>
+          <min>0.2</min>
+          <max>20</max>
           <resolution>0.01</resolution>
         </range>
@@ -137,18 +132,45 @@
   <!-- ===================== Orbbec Astra (Parte 2) ===================== -->
   <!-- TODO: link "camara_link" (caja) con dimensiones y masa de la hoja de datos -->
+  <link name="camara_link">
+      <visual>
+        <origin xyz="0 0 0.02" rpy="0 0 0"/>
+        <geometry><box size="0.040 0.165 0.048"/></geometry>
+        <material name="negro"><color rgba="0.1 0.1 0.1 1"/></material>
+      </visual>
+      <collision>
+        <origin xyz="0 0 0.02" rpy="0 0 0"/>
+        <geometry><box size="0.040 0.165 0.048"/></geometry>
+      </collision>
+      <inertial>
+        <origin xyz="0 0 0.02" rpy="0 0 0"/>
+        <mass value="0.31"/> <!-- Masa kg -->
+        <xacro:inercia_cilindro m="0.31" x="0.040" y="0.165" z="0.048"/>
+      </inertial>
+  </link>
   <!-- TODO: joint fijo "joint_camara" base_link -> camara_link en la posición de su variante -->
+  <joint name="camara_joint" type="fixed">
+    <parent link="base_link"/>
+    <child link="camara_link"/>
+    <origin xyz="0.16 0 0.09" rpy="0 0 0"/>
+  </joint>
   <!-- TODO: link "camara_optica_link" y joint fijo "joint_camara_optica" desde
        camara_link con rpy = (-π/2, 0, -π/2) (REP-103) -->
+  <link name="camara_optica_link"/>
+    <joint name="joint_camara_optica" type="fixed">
+      <parent link="camara_link"/>
+      <child link="camara_optica_link"/>
+      <origin xyz="0 0 0" rpy="${-pi/2} 0 ${-pi/2}"/>
+  </joint>
   <gazebo reference="camara_link">
     <sensor name="astra" type="rgbd_camera">
       <topic>/camara</topic>
-      <gz_frame_id>TODO</gz_frame_id>
-      <update_rate>TODO</update_rate>
+      <gz_frame_id>camara_link</gz_frame_id>
+      <update_rate>30</update_rate>
       <always_on>1</always_on>
       <camera>
-        <horizontal_fov>TODO</horizontal_fov>   <!-- en radianes -->
+        <horizontal_fov>1.01927</horizontal_fov>   <!-- 58.4° en radianes -->
         <image>
-          <width>TODO</width>
-          <height>TODO</height>
+          <width>640</width>
+          <height>480</height>
           <format>R8G8B8</format>
         </image>

Commit message: Examen Parte 3: Bridge configurado y RViz funcionando

File: ros2_ws_mecanum/src/mi_robot_mecanum/urdf/mi_robot.urdf.xacro (robot description, xacro)
@@ -6,7 +6,7 @@
   <!-- ===================== Parámetros de la variante ===================== -->
   <!-- TODO (Parte 1): reemplace cada ${TODO} por el valor de su variante -->
-  <xacro:property name="rueda_radio" value=0.045/>         <!-- r (m) -->
-  <xacro:property name="distancia_ejes" value=0.32/>      <!-- wheelbase (m) -->
-  <xacro:property name="separacion_ruedas" value=0.34/>   <!-- track (m) -->
+  <xacro:property name="rueda_radio" value="0.045"/>         <!-- r (m) -->
+  <xacro:property name="distancia_ejes" value="0.32"/>      <!-- wheelbase (m) -->
+  <xacro:property name="separacion_ruedas" value="0.34"/>   <!-- track (m) -->
   <xacro:property name="lx" value="${distancia_ejes / 2.0}"/>
   <xacro:property name="ly" value="${separacion_ruedas / 2.0}"/>
@@ -71,5 +71,5 @@
       <parent link="base_link"/>
       <child link="rueda_${prefijo}"/>
-      <origin xyz="x_signo*lx, y_signo*ly, 0" rpy="${-pi/2} 0 0"/>
+      <origin xyz="${x_signo*lx} ${y_signo*ly} 0" rpy="${-pi/2} 0 0"/>
       <axis xyz="0 0 1"/>
     </joint>
@@ -84,18 +84,18 @@
        visual, collision e inertial -->
   <link name="lidar_link">
-  <visual>
-    <origin xyz="0 0 0.02" rpy="0 0 0"/>
-    <geometry><cylinder radius="0.038" length="0.041"/></geometry>
-    <material name="negro"><color rgba="0.1 0.1 0.1 1"/></material>
-  </visual>
-  <collision>
-    <origin xyz="0 0 0.02" rpy="0 0 0"/>
-    <geometry><cylinder radius="0.038" length="0.041"/></geometry>
-  </collision>
-  <inertial>
-    <origin xyz="0 0 0.02" rpy="0 0 0"/>
-    <mass value="0.19"/> <!-- Masa kg -->
-    <xacro:inercia_cilindro m="0.19" r="0.038" h="0.041"/>
-  </inertial>
+    <visual>
+      <origin xyz="0 0 0.02" rpy="0 0 0"/>
+      <geometry><cylinder radius="0.038" length="0.041"/></geometry>
+      <material name="negro"><color rgba="0.1 0.1 0.1 1"/></material>
+    </visual>
+    <collision>
+      <origin xyz="0 0 0.02" rpy="0 0 0"/>
+      <geometry><cylinder radius="0.038" length="0.041"/></geometry>
+    </collision>
+    <inertial>
+      <origin xyz="0 0 0.02" rpy="0 0 0"/>
+      <mass value="0.19"/> <!-- Masa kg -->
+      <xacro:inercia_cilindro m="0.19" r="0.038" h="0.041"/>
+    </inertial>
   </link>
   <!-- TODO: joint fijo "joint_lidar" base_link -> lidar_link en la posición de su variante -->
@@ -145,5 +145,5 @@
         <origin xyz="0 0 0.02" rpy="0 0 0"/>
         <mass value="0.31"/> <!-- Masa kg -->
-        <xacro:inercia_cilindro m="0.31" x="0.040" y="0.165" z="0.048"/>
+        <xacro:inercia_caja m="0.31" x="0.040" y="0.165" z="0.048"/>
       </inertial>
   </link>
